File: mixer_module.brd (EAGLE design)
At the start: 80 x 75.9 mm, 85 parts, among them T1 ATB3225-75032CT, T2 ATB3225-75032CT, U2 TS974, U3 TS974, U4 MCP4812

Commit message: final changes to unused external boards
Parts:
- moved R12 3.17 mm to (44.5, 61.6), turned to 0 degrees
- moved C28 2.73 mm to (66.4, 40.3), turned to 180 degrees
- moved C9 2.56 mm to (44.5, 58.1), turned to 180 degrees
- moved C4 1.91 mm to (12.1, 65.4)
- moved C5 1.91 mm to (14.6, 65.4)
- moved C6 1.91 mm to (17.1, 65.4)
- moved C8 1.91 mm to (9.53, 60.3)
- moved R10 1.91 mm to (14.6, 60.3)
- moved R11 1.91 mm to (17.1, 60.3)
- moved R7 1.91 mm to (6.99, 60.3)
- moved R8 1.91 mm to (9.53, 65.4)
- moved R9 1.91 mm to (12.1, 60.3)
- moved C16 1.90 mm to (14.6, 55.2)
- moved R14 1.90 mm to (7.62, 55.2)
- moved R15 1.90 mm to (12.1, 55.2)
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Connections:
- removed net N$76: C6.1, R38.3, TP7.1, U3.8
- new net N$1: C38.1, R37.1, R38.3
- net N$74: now also C6.1, TP7.1, U3.8; no longer C38.1, R37.1
Routing:
- net GND: track 0.00 -> 23.8 mm
- net VCC: track 35.0 -> 49.6 mm
- net AGND: track 22.9 -> 34.8 mm
- net N$76: track 8.37 -> 0.00 mm
- net N$1: track 0.00 -> 6.67 mm
- net N$74: track 12.4 -> 7.45 mm
- net N$75: track 18.9 -> 14.3 mm
- net N$23: track 22.5 -> 24.9 mm
- net N$22: track 18.4 -> 20.3 mm
- net RBDS: track 14.7 -> 13.3 mm
- net N$66: track 13.3 -> 14.5 mm
- net N$42: track 2.99 -> 3.86 mm
- net N$28: track 13.2 -> 12.7 mm
