File: mixer_module.sch (EAGLE design)
At the start: 85 parts, among them T1 ATB3225-75032CT, T2 ATB3225-75032CT, U2 TS974, U3 TS974, U4 MCP4812

Commit message: final changes to unused external boards
Connections:
- removed net N$76: C6.1, R38.E, TP7.1, U3C.OUT
- new net N$1: C38.1, R37.1, R38.E
- net N$74: now also C6.1, TP7.1, U3C.OUT; no longer C38.1, R37.1
Changed lines of the file:
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@@
 <instance part="GND56" gate="1" x="223.52" y="50.8"/>
 <instance part="GND57" gate="1" x="238.76" y="50.8"/>
-<instance part="R38" gate="G$1" x="246.38" y="68.58" rot="R270"/>
+<instance part="R38" gate="G$1" x="246.38" y="68.58" rot="MR270"/>
 <instance part="C6" gate="G$1" x="276.86" y="58.42" rot="R90"/>
 <instance part="AGND5" gate="VR1" x="246.38" y="50.8"/>
@@
 <net name="N$74" class="0">
 <segment>
-<pinref part="R37" gate="G$1" pin="1"/>
-<wire x1="236.22" y1="68.58" x2="238.76" y2="68.58" width="0.1524" layer="91"/>
-<pinref part="C38" gate="G$1" pin="1"/>
-<wire x1="238.76" y1="68.58" x2="241.3" y2="68.58" width="0.1524" layer="91"/>
-<wire x1="238.76" y1="66.04" x2="238.76" y2="68.58" width="0.1524" layer="91"/>
-<junction x="238.76" y="68.58"/>
 <pinref part="R38" gate="G$1" pin="A"/>
-</segment>
-</net>
-<net name="N$75" class="0">
-<segment>
-<wire x1="248.92" y1="60.96" x2="246.38" y2="60.96" width="0.1524" layer="91"/>
-<pinref part="R38" gate="G$1" pin="S"/>
-<wire x1="246.38" y1="60.96" x2="246.38" y2="63.5" width="0.1524" layer="91"/>
-<pinref part="U3" gate="C" pin="-IN"/>
-</segment>
-</net>
-<net name="N$76" class="0">
-<segment>
-<pinref part="R38" gate="G$1" pin="E"/>
 <wire x1="251.46" y1="68.58" x2="266.7" y2="68.58" width="0.1524" layer="91"/>
 <wire x1="266.7" y1="68.58" x2="266.7" y2="58.42" width="0.1524" layer="91"/>
@@
 <pinref part="TP7" gate="G$1" pin="1"/>
 <wire x1="269.24" y1="68.58" x2="266.7" y2="68.58" width="0.1524" layer="91"/>
+</segment>
+</net>
+<net name="N$75" class="0">
+<segment>
+<wire x1="248.92" y1="60.96" x2="246.38" y2="60.96" width="0.1524" layer="91"/>
+<pinref part="R38" gate="G$1" pin="S"/>
+<wire x1="246.38" y1="60.96" x2="246.38" y2="63.5" width="0.1524" layer="91"/>
+<pinref part="U3" gate="C" pin="-IN"/>
 </segment>
 </net>
@@
 </segment>
 </net>
+<net name="N$1" class="0">
+<segment>
+<pinref part="R38" gate="G$1" pin="E"/>
+<pinref part="R37" gate="G$1" pin="1"/>
+<wire x1="236.22" y1="68.58" x2="238.76" y2="68.58" width="0.1524" layer="91"/>
+<wire x1="238.76" y1="68.58" x2="241.3" y2="68.58" width="0.1524" layer="91"/>
+<junction x="238.76" y="68.58"/>
+<pinref part="C38" gate="G$1" pin="1"/>
+<wire x1="238.76" y1="66.04" x2="238.76" y2="68.58" width="0.1524" layer="91"/>
+</segment>
+</net>
