File: vco_module.brd (EAGLE design)
At the start: 14.3 x 26.3 mm, 11 parts, among them U1 MAX2606

Commit message: fixed for boardmill
Parts:
- moved L1 1.27 mm to (2.22, 10.2)
- moved JP2 0.32 mm to (4.76, 2.54)
Routing:
- net N$24: track 1.99 -> 3.26 mm
Changed lines of the file:
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@@
 <vertex x="6.35" y="11.43"/>
 <vertex x="6.35" y="8.89"/>
-<vertex x="3.81" y="8.89"/>
-<vertex x="3.81" y="11.43"/>
+<vertex x="5.08" y="8.89"/>
+<vertex x="5.08" y="11.43"/>
+</polygon>
+<polygon width="0.4064" layer="41">
+<vertex x="8.89" y="9.525"/>
+<vertex x="12.3825" y="9.525"/>
+<vertex x="12.3825" y="10.795"/>
+<vertex x="8.89" y="10.795"/>
+</polygon>
+<polygon width="0.4064" layer="41">
+<vertex x="4.445" y="18.415"/>
+<vertex x="8.255" y="18.415"/>
+<vertex x="8.255" y="19.685"/>
+<vertex x="4.445" y="19.685"/>
+</polygon>
+<polygon width="0.6096" layer="41">
+<vertex x="2.8575" y="10.4775"/>
+<vertex x="2.8575" y="8.5725"/>
+<vertex x="1.5875" y="8.5725"/>
+<vertex x="1.5875" y="10.4775"/>
 </polygon>
 </plain>
@@
 <attribute name="VALUE" x="4.445" y="6.985" size="1.27" layer="27"/>
 </element>
-<element name="L1" library="resistor" package="L3216C" value="485nH" x="3.4925" y="10.16" smashed="yes" rot="R270">
-<attribute name="NAME" x="2.032" y="11.4935" size="1.016" layer="25" font="vector" rot="R90"/>
-<attribute name="VALUE" x="1.0795" y="11.684" size="1.27" layer="27" rot="R270"/>
+<element name="L1" library="resistor" package="L3216C" value="485nH" x="2.2225" y="10.16" smashed="yes" rot="R270">
+<attribute name="NAME" x="0.762" y="11.4935" size="1.016" layer="25" font="vector" rot="R90"/>
+<attribute name="VALUE" x="-0.1905" y="11.684" size="1.27" layer="27" rot="R270"/>
 </element>
 <element name="C10" library="adafruit" package="C1206" value="1uF" x="9.2075" y="10.16" smashed="yes" rot="R270">
@@
 </element>
 <element name="JP1" library="sparkfun" package="1X02" value="" x="5.08" y="24.13"/>
-<element name="JP2" library="sparkfun" package="1X03" value="" x="5.08" y="2.54"/>
+<element name="JP2" library="sparkfun" package="1X03" value="" x="4.7625" y="2.54"/>
 </elements>
 <signals>
@@
 <contactref element="U1" pad="1"/>
 <contactref element="L1" pad="2"/>
-<wire x1="5.4" y1="8.86" x2="3.84" y2="8.86" width="0.6096" layer="1"/>
-<wire x1="3.84" y1="8.86" x2="3.81" y2="8.89" width="0.4064" layer="1"/>
-<wire x1="3.81" y1="8.89" x2="3.4925" y2="8.66" width="0.4064" layer="1"/>
+<wire x1="5.4" y1="8.86" x2="2.57" y2="8.86" width="0.6096" layer="1"/>
+<wire x1="2.57" y1="8.86" x2="2.54" y2="8.89" width="0.4064" layer="1"/>
+<wire x1="2.54" y1="8.89" x2="2.2225" y2="8.66" width="0.4064" layer="1"/>
 </signal>
 <signal name="N$33">
@@
 <wire x1="7.3" y1="6.67" x2="7.62" y2="6.35" width="0.4064" layer="1"/>
 <contactref element="JP2" pad="1"/>
-<wire x1="5.08" y1="2.54" x2="5.08" y2="3.81" width="0.6096" layer="1"/>
-<wire x1="5.08" y1="3.81" x2="7.62" y2="6.35" width="0.6096" layer="1"/>
 <wire x1="7.62" y1="6.22" x2="7.62" y2="6.35" width="0.4064" layer="1"/>
+<wire x1="7.62" y1="6.22" x2="7.49" y2="6.22" width="0.6096" layer="1"/>
+<wire x1="7.49" y1="6.22" x2="4.7625" y2="3.4925" width="0.6096" layer="1"/>
+<wire x1="4.7625" y1="2.54" x2="4.7625" y2="3.4925" width="0.6096" layer="1"/>
 </signal>
 <signal name="VCC">
@@
 <wire x1="11.43" y1="11.56" x2="11.43" y2="11.43" width="0.4064" layer="1"/>
 <contactref element="JP2" pad="3"/>
-<wire x1="10.16" y1="2.54" x2="13.335" y2="5.715" width="0.6096" layer="1"/>
 <wire x1="13.335" y1="5.715" x2="13.335" y2="11.1125" width="0.6096" layer="1"/>
 <wire x1="11.7475" y1="11.56" x2="12.8875" y2="11.56" width="0.6096" layer="1"/>
 <wire x1="12.8875" y1="11.56" x2="13.335" y2="11.1125" width="0.6096" layer="1"/>
+<wire x1="9.8425" y1="2.54" x2="10.16" y2="2.54" width="0.6096" layer="1"/>
+<wire x1="10.16" y1="2.54" x2="13.335" y2="5.715" width="0.6096" layer="1"/>
 </signal>
 </signals>

Commit message: final changes to unused external boards
Parts:
- C10, C11, C15, C2, C3: device adafruit:C1206 -> adafruit:C050-025X075
- JP1: device sparkfun:1X02 -> sparkfun:SCREWTERMINAL-3.5MM-2
- L1: device resistor:L3216C -> resistor:0204V
- R3, R4: device adafruit:R1206 -> adafruit:0207/10
- moved L1 13.3 mm to (15.6, 10.2), turned to 90 degrees
- moved R3 12.2 mm to (14.6, 20.3), turned to 270 degrees
- moved R4 7.89 mm to (3.17, 20.3), turned to 270 degrees
- moved JP1 6.61 mm to (10.5, 27.9), turned to 180 degrees
- moved C2 5.85 mm to (10.8, 20.3)
- moved C15 5.12 mm to (4.45, 8.89), turned to 270 degrees
- moved U1 4.58 mm to (8.89, 14.0), flipped to the bottom
- moved C11 4.42 mm to (10.2, 6.03), turned to 180 degrees
- moved C3 1.42 mm to (6.99, 20.3)
- moved JP2 1.27 mm to (6.03, 2.54)
- moved C10 1.00 mm to (10.2, 9.84), turned to 180 degrees
Routing:
- net VCC: track 25.7 -> 50.7 mm
- net SIGNAL: track 10.5 -> 13.6 mm
- net N$24: track 3.26 -> 6.23 mm
- net N$39: track 3.68 -> 5.21 mm
- net N$52: track 3.68 -> 5.08 mm
- net N$35: track 9.17 -> 7.77 mm
- net N$33: track 9.17 -> 7.77 mm
- net GND: track 0.92 -> 0.00 mm
- added copper zone on layer 16, net GND
- added copper zone on layer 16, net N$1
- removed copper zone on layer 1, net GND
Other:
- board size 14.3 x 26.3 mm -> 18.1 x 31.4 mm
